File: PCB/speedcoach.kicad_pcb (KiCad board)
At the start: 2 copper layers, 0 parts

Commit message: placement
Parts:
- added C1: 4.7uF, Capacitor_SMD:C_0805_2012Metric, F.Cu at (115.2, 118.2)
- added C10: 100nF, Capacitor_SMD:C_0805_2012Metric, F.Cu at (126.5, 85.1)
- added C2: 4.3pF, Capacitor_SMD:C_0805_2012Metric, F.Cu at (126.5, 103.6)
- added C3: 4.3pF, Capacitor_SMD:C_0805_2012Metric, F.Cu at (119.4, 103.6)
- added C4: 4.7uF, Capacitor_SMD:C_0805_2012Metric, F.Cu at (111.9, 118.2)
- added C5: 100nF, Capacitor_SMD:C_0805_2012Metric, F.Cu at (119.4, 85.1)
- added C6: 100nF, Capacitor_SMD:C_0805_2012Metric, F.Cu at (115.8, 98.6)
- added C7: 100nF, Capacitor_SMD:C_0805_2012Metric, F.Cu at (129.8, 85.1)
- added C8: 100nF, Capacitor_SMD:C_0805_2012Metric, F.Cu at (130.0, 103.6)
- added C9: 100nF, Capacitor_SMD:C_0805_2012Metric, F.Cu at (115.8, 103.6)
- added J1: Conn_01x04_Male, Connector_PinHeader_2.54mm:PinHeader_1x04_P2.54mm_Horizontal, B.Cu at (159.3, 111.4)
- added J2: Conn_01x04_Male, Connector_PinHeader_2.54mm:PinHeader_1x04_P2.54mm_Horizontal, B.Cu at (156.7, 77.5)
- added J3: Conn_01x04_Male, Connector_PinHeader_2.54mm:PinHeader_1x04_P2.54mm_Horizontal, B.Cu at (118.6, 77.5)
- added J4: USB_B_Micro, speedcoach:10118194-0001LF, F.Cu at (113.5, 125.3)
- added J5: 440055-2, speedcoach:440055-2, F.Cu at (156.9, 121.3)
- added R1: 220, Resistor_SMD:R_0805_2012Metric, F.Cu at (146.6, 124.2)
- added R10: 3k3, Resistor_SMD:R_0805_2012Metric, F.Cu at (112.3, 103.7)
- added R11: 3k3, Resistor_SMD:R_0805_2012Metric, F.Cu at (112.3, 93.5)
- added R12: 3k3, Resistor_SMD:R_0805_2012Metric, F.Cu at (112.3, 85.1)
- added R2: 10k, Resistor_SMD:R_0805_2012Metric, F.Cu at (140.6, 124.2)
- added R3: NP, Resistor_SMD:R_0805_2012Metric, F.Cu at (134.5, 108.0)
- added R4: 10k, Resistor_SMD:R_0805_2012Metric, F.Cu at (134.6, 124.2)
- added R5: 3k3, Resistor_SMD:R_0805_2012Metric, F.Cu at (140.5, 108.0)
- added R6: 3k3, Resistor_SMD:R_0805_2012Metric, F.Cu at (146.4, 108.0)
- added R7: 2k, Resistor_SMD:R_0805_2012Metric, F.Cu at (118.5, 118.2)
- added R8: 10k, Resistor_SMD:R_0805_2012Metric, F.Cu at (108.6, 118.2)
- added R9: 10k, Resistor_SMD:R_0805_2012Metric, F.Cu at (115.8, 93.5)
- added SW1: 1825027-8, speedcoach:1825027-8, F.Cu at (105.3, 108.2)
- added SW2: 1825027-8, speedcoach:1825027-8, F.Cu at (105.3, 96.5)
- added SW3: 1825027-8, speedcoach:1825027-8, F.Cu at (105.3, 84.9)
- added U1: PA1010D, speedcoach:PA1010D, F.Cu at (122.4, 111.3)
- added U2: DA14531MOD, speedcoach:DA14531MOD-00F01002, F.Cu at (163.1, 87.3)
- added U3: ORG1411-PM04, speedcoach:ORG1411, F.Cu at (140.2, 116.3)
- added U4: GLCD_2.7INCH, speedcoach:SHARP_DISPLAY_400x240, F.Cu at (102.2, 126.4)
- added U5: PIM456, speedcoach:PIM456, F.Cu at (153.9, 103.8)
- added U6: Bluefruit, speedcoach:Bluefruit, F.Cu at (142.5, 78.2)
- added U7: MB85RS256TY, Package_SO:SOP-8_3.9x4.9mm_P1.27mm, F.Cu at (127.1, 79.0)
- added U8: MCP73831, speedcoach:MCP73831T-2ATIOT, F.Cu at (115.2, 112.1)
- added U9: STM32L051C8T3, Package_QFP:LQFP-48_7x7mm_P0.5mm, F.Cu at (124.2, 93.6)
- added XTAL1: NX3215SA-32.768K, speedcoach:NX3215SA-32.768K-EXS00A-MU00003, F.Cu at (122.9, 103.3)
Routing:
- net +3V3: track 0.00 -> 47.6 mm
- net GND: track 0.00 -> 40.0 mm
- net Net-(U9-PC14-OSC32_IN): track 0.00 -> 11.2 mm
- net Net-(U9-PC15-OSC32_OUT): track 0.00 -> 8.15 mm
Other:
- board outline added: 64.5 x 56.9 mm

Commit message: routed v1
Parts:
- moved R5 15.5 mm to (130.7, 120.0), turned to 0 degrees
- moved R2 9.61 mm to (149.2, 120.0), turned to 0 degrees
- moved R4 8.62 mm to (130.7, 116.5), turned to 180 degrees
- moved R1 8.07 mm to (149.2, 116.6)
- moved R3 6.34 mm to (130.7, 113.0), turned to 0 degrees
- moved R6 5.91 mm to (149.2, 113.2), turned to 180 degrees
- moved R12 0.76 mm to (113.0, 85.1)
- moved U3 0.63 mm to (139.6, 116.3)
- turned C4 to -90 degrees
- turned R8 to 90 degrees
Connections:
- J1 pad 2: BLE_UART_RX -> BLE_UART_TX
- J1 pad 3: BLE_UART_TX -> BLE_UART_RX
- J2 pad 2: /GPS, Acceleromter, BLE, GLCD/BLE_SWCLK -> /GPS, Acceleromter, BLE, GLCD/BLE_SWDIO
- J2 pad 3: /GPS, Acceleromter, BLE, GLCD/BLE_SWDIO -> /GPS, Acceleromter, BLE, GLCD/BLE_SWCLK
Routing:
- net BLE_UART_TX: track 0.00 -> 89.7 mm, vias 0 -> 3
- net BLE_UART_RX: track 0.00 -> 76.2 mm, vias 0 -> 5
- net BLE_ACCEL_SCL: track 0.00 -> 70.0 mm, vias 0 -> 3
- net GPS_SCL: track 0.00 -> 64.3 mm, vias 0 -> 3
- net BLE_ACCEL_SDA: track 0.00 -> 57.3 mm
- net GND: track 40.0 -> 90.6 mm, vias 0 -> 16
- net ACCEL_INT: track 0.00 -> 48.3 mm, vias 0 -> 2
- net +3V3: track 47.6 -> 90.2 mm, vias 0 -> 15
- net GPS_SDA: track 0.00 -> 42.3 mm, vias 0 -> 1
- net BLE_RST: track 0.00 -> 41.2 mm, vias 0 -> 2
- net GPS_ONOFF: track 0.00 -> 34.8 mm, vias 0 -> 2
- net GPS_1PPS: track 0.00 -> 34.6 mm, vias 0 -> 2
- net BTN_UP: track 0.00 -> 33.7 mm, vias 0 -> 2
- net LCD_CS: track 0.00 -> 30.6 mm, vias 0 -> 1
- net BTN_DWN: track 0.00 -> 30.4 mm
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- added copper zone on In1.Cu, net +3V3
- added copper zone on In2.Cu, net GND
Other:
- copper layers 2 -> 4
