File: PCB/speedcoach/speedcoach.kicad_pcb (KiCad board)
At the start: 2 copper layers, 64.8 x 57.1 mm, 40 parts, among them J1 Conn_01x04_Male, J2 Conn_01x04_Male, J3 Conn_01x04_Male, J4 USB_B_Micro, J5 440055-2, SW1 1825027-8, SW2 1825027-8, SW3 1825027-8, U1 PA1010D, U2 DA14531MOD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

Commit message: added 3D models
Parts:
- J3: moved to B.Cu
- J5: moved to F.Cu
- moved J5 1.76 mm to (164.8, 111.6), turned to -90 degrees
- moved C4 0.52 mm to (160.8, 112.5), turned to 90 degrees
- turned J3 to 0 degrees
Routing:
- net +3V3: track 85.7 -> 86.3 mm

Commit message: optimization
Parts:
- J5: value 440055-2 -> CONN_440055-2_TEC
- SW1, SW2, SW3: value 1825027-8 -> SW2_1825027-C_TEC
Routing:
- net CHARGE_STATUS: track 48.0 -> 45.9 mm, vias 3 -> 2
- net /MCU, Charger, Buttons/MCU_SWCLK: track 11.5 -> 10.8 mm
- net BTN_ENTER: track 41.8 -> 42.5 mm
- net Net-(C1-Pad1): track 17.5 -> 16.9 mm
